Commit message: modified d435 visual stl model to be positioned 1 cm backwards

File: realsense2_description/urdf/_d435.urdf.xacro (robot description, xacro)
@@ -22,5 +22,5 @@
     <xacro:property name="d435_cam_height" value="0.025"/>
     <xacro:property name="d435_cam_depth" value="0.02505"/>
-    <xacro:property name="d435_cam_mount_from_center_offset" value="0.0149"/>
+    <xacro:property name="d435_cam_mount_from_center_offset" value="0.01"/>
     <!-- The following offset is relative the the physical D435 camera peripherial
   	camera tripod mount -->
